Commit message: Add unitree lidar to robot model

File: officebot_description/urdf/officebot.xacro (robot description, xacro)
@@ -55,5 +55,5 @@
     </joint>
     <!-- Lidar -->
-    <link name="rplidar_link">
+    <link name="unilidar_lidar">
         <inertial>
             <origin xyz="0 0 0" rpy="0 0 0" />
@@ -76,7 +76,8 @@
     </link>
     <joint name="joint_sensor_laser" type="fixed">
-        <origin xyz="0 0 0.120" rpy="0 0 ${PI}"/>
+    <!-- ${PI} -->
+        <origin xyz="0.130 0.0 0.214" rpy="0 ${PI * 0.25} 0"/>
         <parent link="body_link"/>
-        <child link="rplidar_link"/>
+        <child link="unilidar_lidar"/>
     </joint>
     <!-- Camera-->

Commit message: Correct lidar position

File: officebot_description/urdf/officebot.xacro (robot description, xacro)
@@ -76,6 +76,6 @@
     </link>
     <joint name="joint_sensor_laser" type="fixed">
-    <!-- ${PI} -->
-        <origin xyz="0.130 0.0 0.214" rpy="0 ${PI * 0.25} 0"/>
+    <!-- ${PI} ${PI * -0.375} -->
+	    <origin xyz="0.130 0.0 0.214" rpy="0 ${PI * 0.25} 0"/>
         <parent link="body_link"/>
         <child link="unilidar_lidar"/>

Commit message: Fix lidar height

File: officebot_description/urdf/officebot.xacro (robot description, xacro)
@@ -77,5 +77,5 @@
     <joint name="joint_sensor_laser" type="fixed">
     <!-- ${PI} ${PI * -0.375} -->
-	    <origin xyz="0.130 0.0 0.214" rpy="0 ${PI * 0.25} 0"/>
+	    <origin xyz="0.130 0.0 0.15565" rpy="0 ${PI * 0.25} 0"/>
         <parent link="body_link"/>
         <child link="unilidar_lidar"/>

Commit message: Update robot model

File: officebot_description/urdf/officebot.xacro (robot description, xacro)
@@ -32,12 +32,19 @@
 			<origin xyz="0 0 -0.015" rpy="${PI/2} 0 ${PI/2}" />
             <geometry>
-                <mesh filename="package://officebot_description/meshes/officebot_body_link.stl" scale="0.001 0.001 0.001" />
-            </geometry>
-			<material name="White" />
+                <mesh filename="package://officebot_description/meshes/officebot_body_bottom.stl" scale="0.001 0.001 0.001" />
+            </geometry>
+			<material name="Grey" />
+		</visual>
+		<visual>
+			<origin xyz="0 0 0.085" rpy="${PI/2} 0 ${PI/2}" />
+            <geometry>
+                <mesh filename="package://officebot_description/meshes/officebot_body_top.stl" scale="0.001 0.001 0.001" />
+            </geometry>
+			<material name="Red" />
 		</visual>
 		<collision>
 			<origin xyz="0 0 -0.015" rpy="${PI/2} 0 ${PI/2}" />
             <geometry>
-                <mesh filename="package://officebot_description/meshes/officebot_body_link.stl" scale="0.001 0.001 0.001" />
+                <mesh filename="package://officebot_description/meshes/officebot_body_bottom.stl" scale="0.001 0.001 0.001" />
             </geometry>
 		</collision>
@@ -77,5 +84,5 @@
     <joint name="joint_sensor_laser" type="fixed">
     <!-- ${PI} ${PI * -0.375} -->
-	    <origin xyz="0.130 0.0 0.15565" rpy="0 ${PI * 0.25} 0"/>
+	    <origin xyz="0.145 0.0 0.17665" rpy="0 ${PI * 0.25} 0"/>
         <parent link="body_link"/>
         <child link="unilidar_lidar"/>
@@ -108,5 +115,31 @@
         <parent link="body_link"/>
         <child link="camera_link"/>
-        <origin xyz="0.330 0 0.035" rpy="0 0 0"/>
+        <origin xyz="0.175 0 0.100" rpy="0 0 0"/>
+    </joint>
+    <!-- IMU -->
+    <link name="unilidar_imu">
+        <inertial>
+            <origin xyz="0 0 0" rpy="0 0 0" />
+            <mass value="0.1" />
+            <inertia ixx="0.0" ixy="0.0" ixz="0.0" iyy="0.0" iyz="0.0" izz="0.0" />
+        </inertial>
+        <visual>
+            <origin xyz="0 0 0" rpy="0 0 0" />
+            <geometry>
+                <box size="0.010 0.010 0.010" />
+            </geometry>
+            <material name="Green" />
+        </visual>
+        <collision>
+            <origin xyz="0 0 0" rpy="0 0 0"/>
+            <geometry>
+                <box size="0.010 0.010 0.010" />
+            </geometry>
+        </collision>
+    </link>
+    <joint name="joint_sensor_imu" type="fixed">
+        <parent link="unilidar_lidar"/>
+        <child link="unilidar_imu"/>
+        <origin xyz="0 0 0" rpy="0 0 0"/>
     </joint>
     <!-- Wheels -->
@@ -117,5 +150,5 @@
                 <cylinder length="${wheel_width}" radius="${wheel_radius}"/>
             </geometry>
-            <material name="Red" />
+            <material name="Black" />
         </visual>
         <collision>
@@ -149,5 +182,5 @@
                 <cylinder length="${wheel_width}" radius="${wheel_radius}"/>
             </geometry>
-            <material name="Red" />
+            <material name="Black" />
         </visual>
         <collision>
@@ -181,5 +214,5 @@
                 <cylinder length="${wheel_width}" radius="${wheel_radius}"/>
             </geometry>
-            <material name="Red" />
+            <material name="Black" />
         </visual>
         <collision>
@@ -213,5 +246,5 @@
                 <cylinder length="${wheel_width}" radius="${wheel_radius}"/>
             </geometry>
-            <material name="Red" />
+            <material name="Black" />
         </visual>
         <collision>

File: officebot_description/urdf/officebot_materials.xacro (robot description, xacro)
@@ -14,4 +14,7 @@
 		<color rgba="1.0 1.0 1.0 1.0"/>
 	</material>
+	<material name="Grey">
+		<color rgba="0.5 0.5 0.5 1.0"/>
+	</material>
 	<material name="Black">
 		<color rgba="0.0 0.0 0.0 1.0"/>

Commit message: Update wheel separation

File: officebot_description/urdf/officebot.xacro (robot description, xacro)
@@ -9,5 +9,5 @@
     <xacro:property name="body_height" value="0.17" />
     <xacro:property name="wheel_radius" value="0.05835"/>
-    <xacro:property name="wheel_separation" value="0.20"/>
+    <xacro:property name="wheel_separation" value="0.243"/>
     <xacro:property name="wheel_distance" value="0.125"/>
     <xacro:property name="wheel_width" value="0.043"/>

Commit message: Update robot model

File: officebot_description/urdf/officebot.xacro (robot description, xacro)
@@ -62,5 +62,5 @@
     </joint>
     <!-- Lidar -->
-    <link name="unilidar_lidar">
+    <!-- <link name="unilidar_lidar">
         <inertial>
             <origin xyz="0 0 0" rpy="0 0 0" />
@@ -79,4 +79,24 @@
             <geometry>
                 <cylinder radius="0.035" length="0.025"/>
+            </geometry>
+        </collision>
+    </link> -->
+    <link name="laser">
+        <inertial>
+            <origin xyz="0 0 0" rpy="0 0 0" />
+            <mass value="0.1" />
+            <inertia ixx="0.0" ixy="0.0" ixz="0.0" iyy="0.0" iyz="0.0" izz="0.0" />
+        </inertial>
+        <visual>
+            <origin xyz="0 0 0" rpy="0 0 0" />
+            <geometry>
+                <cylinder radius="0.036" length="0.021"/>
+            </geometry>
+            <material name="Blue" />
+        </visual>
+        <collision>
+            <origin xyz="0 0 0" rpy="0 0 0"/>
+            <geometry>
+                <cylinder radius="0.036" length="0.021"/>
             </geometry>
         </collision>
@@ -84,7 +104,7 @@
     <joint name="joint_sensor_laser" type="fixed">
     <!-- ${PI} ${PI * -0.375} -->
-	    <origin xyz="0.145 0.0 0.17665" rpy="0 ${PI * 0.25} 0"/>
+	    <origin xyz="0.100 0.0 0.235" rpy="0 0 0"/>
         <parent link="body_link"/>
-        <child link="unilidar_lidar"/>
+        <child link="laser"/>
     </joint>
     <!-- Camera-->
@@ -118,5 +138,5 @@
     </joint>
     <!-- IMU -->
-    <link name="unilidar_imu">
+    <!-- <link name="unilidar_imu">
         <inertial>
             <origin xyz="0 0 0" rpy="0 0 0" />
@@ -137,10 +157,36 @@
             </geometry>
         </collision>
-    </link>
-    <joint name="joint_sensor_imu" type="fixed">
+    </link> -->
+    <!-- <joint name="joint_sensor_imu" type="fixed">
         <parent link="unilidar_lidar"/>
         <child link="unilidar_imu"/>
         <origin xyz="0 0 0" rpy="0 0 0"/>
-    </joint>
+    </joint> -->
+    <!-- rear lidar -->
+    <!-- <link name="ydlidar1">
+        <inertial>
+            <origin xyz="0 0 0" rpy="0 0 0" />
+            <mass value="0.1" />
+            <inertia ixx="0.0" ixy="0.0" ixz="0.0" iyy="0.0" iyz="0.0" izz="0.0" />
+        </inertial>
+        <visual>
+            <origin xyz="0 0 0" rpy="0 0 0" />
+            <geometry>
+                <box size="0.010 0.010 0.010" />
+            </geometry>
+            <material name="Green" />
+        </visual>
+        <collision>
+            <origin xyz="0 0 0" rpy="0 0 0"/>
+            <geometry>
+                <box size="0.000 0.000 0.000" />
+            </geometry>
+        </collision>
+    </link> -->
+    <!-- <joint name="joint_sensor_ydlidar1" type="fixed">
+        <parent link="body_link"/>
+        <child link="ydlidar1"/>
+        <origin xyz="-0.175 0 0.100" rpy="0 0 ${PI}"/>
+    </joint> -->
     <!-- Wheels -->
     <link name="rear_left_wheel">
@@ -276,5 +322,5 @@
         <parent link="body_link" />
         <child link="rear_left_wheel" />
-        <origin xyz="-${wheel_distance} ${wheel_separation/2 + wheel_width/2} 0" rpy="0 0 0"/>
+        <origin xyz="-${wheel_distance} ${wheel_separation/2} 0" rpy="0 0 0"/>
         <dynamics damping="0.0" friction="0.0"/>
         <limit effort= "100" velocity="100"/>
@@ -284,5 +330,5 @@
         <parent link="body_link" />
         <child link="rear_right_wheel" />
-		<origin xyz="-${wheel_distance} ${-1 * (wheel_separation/2 + wheel_width/2)} 0" rpy="0 0 0"/>
+		<origin xyz="-${wheel_distance} ${-1 * (wheel_separation/2)} 0" rpy="0 0 0"/>
         <dynamics damping="0.0" friction="0.0"/>
         <limit effort= "100" velocity="100"/>
@@ -292,5 +338,5 @@
         <parent link="body_link" />
         <child link="front_left_wheel" />
-		<origin xyz="${wheel_distance} ${wheel_separation/2 + wheel_width/2} 0" rpy="0 0 0" />
+		<origin xyz="${wheel_distance} ${wheel_separation/2} 0" rpy="0 0 0" />
         <dynamics damping="0.0" friction="0.0"/>
         <limit effort= "100" velocity="100"/>
@@ -300,5 +346,5 @@
         <parent link="body_link" />
         <child link="front_right_wheel" />
-		<origin xyz="${wheel_distance} ${-1 * (wheel_separation/2 + wheel_width/2)} 0" rpy="0 0 0" />
+		<origin xyz="${wheel_distance} ${-1 * (wheel_separation/2)} 0" rpy="0 0 0" />
         <dynamics damping="0.0" friction="0.0"/>
         <limit effort= "100" velocity="100"/>

Commit message: Fix robot turning odometry

File: officebot_description/urdf/officebot.xacro (robot description, xacro)
@@ -8,5 +8,5 @@
     <xacro:property name="clearance" value="0.100" />
     <xacro:property name="body_height" value="0.17" />
-    <xacro:property name="wheel_radius" value="0.05835"/>
+    <xacro:property name="wheel_radius" value="0.05035"/>
     <xacro:property name="wheel_separation" value="0.243"/>
     <xacro:property name="wheel_distance" value="0.125"/>

Commit message: Add IMU

File: officebot_description/urdf/officebot.xacro (robot description, xacro)
@@ -108,4 +108,30 @@
         <child link="laser"/>
     </joint>
+    <!-- IMU -->
+    <link name="imu">
+        <inertial>
+            <origin xyz="0 0 0" rpy="0 0 0" />
+            <mass value="0.1" />
+            <inertia ixx="0.0" ixy="0.0" ixz="0.0" iyy="0.0" iyz="0.0" izz="0.0" />
+        </inertial>
+        <visual>
+            <origin xyz="0 0 0" rpy="0 0 0" />
+            <geometry>
+                <box size="0.016 0.016 0.005" />
+            </geometry>
+            <material name="Blue" />
+        </visual>
+        <collision>
+            <origin xyz="0 0 0" rpy="0 0 0"/>
+            <geometry>
+                <box size="0.016 0.016 0.005" />
+            </geometry>
+        </collision>
+    </link>
+    <joint name="joint_imu" type="fixed">
+	    <origin xyz="0.0 0.0 0.062" rpy="0 0 0"/>
+        <parent link="body_link"/>
+        <child link="imu"/>
+    </joint>
     <!-- Camera-->
     <link name="camera_link">
